Commit message: update hexar urdf

File: hexar_description/urdf/hexar.xacro (robot description, xacro)
@@ -1,4 +1,4 @@
 <?xml version="1.0"?>
-<robot xmlns:xacro="http://www.ros.org/wiki/xacro" name="hexar">
+<robot name="hexar" xmlns:xacro="https://www.ros.org/wiki/xacro">
     <!-- Refer to Nav2's URDF tutorial -->
     <!-- https://navigation.ros.org/setup_guides/urdf/setup_urdf.html -->
@@ -13,10 +13,4 @@
         <color rgba="0.3098 0.1765 0.4980 1" />
     </material>
-    <material name="orange">
-        <color rgba="1 0.6471 0 1" />
-    </material>
-    <material name="navy">
-        <color rgba="0 0 0.5 1" />
-    </material>
     <material name="gray">
         <color rgba="0.5 0.5 0.5 1" />
@@ -27,8 +21,8 @@
     <!-- base properties -->
     <xacro:property name="base_radius" value="0.1" />
-    <xacro:property name="base_length" value="0.009" />
+    <xacro:property name="base_height" value="0.009" />
     <xacro:property name="base_mass" value="3" />
     <!-- wheel properties -->
-    <xacro:property name="wheel_xoff" value="0.1" />
+    <xacro:property name="wheel_xoff" value="0.035" />
     <xacro:property name="wheel_yoff" value="0.095" />
     <xacro:property name="wheel_zoff" value="0.009" />
@@ -44,11 +38,11 @@
     <xacro:property name="lidar_radius" value="0.035" />
     <xacro:property name="lidar_height" value="0.02" />
-    <xacro:property name="lidar_zoff" value="0.111" />
+    <xacro:property name="lidar_zoff" value="0.1" />
     <xacro:property name="lidar_mass" value="0.17" />
     <!-- imu properties -->
-    <xacro:property name="imu_width" value="0.02" />
-    <xacro:property name="imu_depth" value="0.015" />
-    <xacro:property name="imu_height" value="0.001" />
-    <xacro:property name="imu_mass" value="0.002" />
+    <!-- <xacro:property name="imu_width" value="0.02" /> -->
+    <!-- <xacro:property name="imu_depth" value="0.015" /> -->
+    <!-- <xacro:property name="imu_height" value="0.001" /> -->
+    <!-- <xacro:property name="imu_mass" value="0.002" /> -->
     <!-- Define intertial property macros  -->
     <xacro:macro name="box_inertia" params="m w d h">
@@ -77,5 +71,5 @@
             <parent link="base_link" />
             <child link="${prefix}_link" />
-            <origin xyz="${wheel_xoff} ${y_reflect*(base_depth/2+wheel_ygap+wheel_width/2)} 0" rpy="${-PI/2} 0 0" />
+            <origin xyz="${wheel_xoff} ${y_reflect * wheel_yoff} ${wheel_zoff}" rpy="${-PI/2} 0 0" />
             <axis xyz="0 0 1" />
         </joint>
@@ -99,11 +93,11 @@
         <visual>
             <geometry>
-                <cylinder length="${base_radius}" radius="${base_length}"/>
-            </geometry>
-            <material name="orange" />
+                <cylinder length="${base_height}" radius="${base_radius}" />
+            </geometry>
+            <material name="white" />
         </visual>
         <collision>
             <geometry>
-                <cylinder length="${base_radius}" radius="${base_length}"/>
+                <cylinder length="${base_height}" radius="${base_radius}" />
             </geometry>
         </collision>
@@ -113,5 +107,5 @@
         <parent link="base_link" />
         <child link="base_footprint" />
-        <origin xyz="0.0 0.0 ${-(wheel_radius)}" rpy="0 0 0" />
+        <origin xyz="0.0 0.0 ${wheel_zoff-wheel_radius}" rpy="0 0 0" />
     </joint>
     <link name="base_footprint" />
@@ -123,24 +117,14 @@
     </joint>
     <link name="base_inertial">
-        <xacro:box_inertia m="${base_mass}" w="${base_width}" d="${base_depth}" h="${base_height}" />
+        <xacro:cylinder_inertia m="${base_mass}" r="${base_radius}" h="${base_height}" />
     </link>
     <!-- Wheels -->
     <xacro:wheel prefix="left_wheel" y_reflect="1" />
-    <gazebo reference="left_wheel_link">
-        <mu1>1.0</mu1>
-        <mu2>1.0</mu2>
-        <material>Gazebo/Blue</material>
-    </gazebo>
     <xacro:wheel prefix="right_wheel" y_reflect="-1" />
-    <gazebo reference="right_wheel_link">
-        <mu1>1.0</mu1>
-        <mu2>1.0</mu2>
-        <material>Gazebo/Blue</material>
-    </gazebo>
     <!-- Caster ball -->
     <joint name="caster_joint" type="fixed">
         <parent link="base_link" />
         <child link="caster" />
-        <origin xyz="${caster_xoff} 0.0 ${-(base_height/2)}" rpy="0 0 0" />
+        <origin xyz="${caster_xoff} 0.0 ${caster_zoff}" rpy="0 0 0" />
     </joint>
     <link name="caster">
@@ -158,9 +142,4 @@
         <xacro:sphere_inertia m="${caster_mass}" r="${caster_radius}" />
     </link>
-    <gazebo reference="caster">
-        <mu1>0.0</mu1>
-        <mu2>0.0</mu2>
-        <material>Gazebo/Gray</material>
-    </gazebo>
     <!-- lidar -->
     <joint name="lidar_joint" type="fixed">
@@ -175,5 +154,5 @@
                 <cylinder radius="${lidar_radius}" length="${lidar_height}" />
             </geometry>
-            <material name="black" />
+            <material name="purple" />
         </visual>
         <collision>
@@ -185,150 +164,93 @@
         <xacro:cylinder_inertia m="${lidar_mass}" r="${lidar_radius}" h="${lidar_height}" />
     </link>
-    <gazebo reference="lidar_link">
-        <material>Gazebo/Black</material>
-        <sensor name="lidar" type="ray">
-            <always_on>true</always_on>
-            <visualize>true</visualize>
-            <update_rate>5</update_rate>
-            <ray>
-                <scan>
-                    <horizontal>
-                        <samples>360</samples>
-                        <resolution>1.000000</resolution>
-                        <min_angle>0.000000</min_angle>
-                        <max_angle>6.280000</max_angle>
-                    </horizontal>
-                </scan>
-                <range>
-                    <min>0.120000</min>
-                    <max>6</max>
-                    <resolution>0.015000</resolution>
-                </range>
-                <noise>
-                    <type>gaussian</type>
-                    <mean>0.0</mean>
-                    <stddev>0.01</stddev>
-                </noise>
-            </ray>
-            <plugin name="scan" filename="libgazebo_ros_ray_sensor.so">
-                <ros>
-                    <remapping>~/out:=scan</remapping>
-                </ros>
-                <output_type>sensor_msgs/LaserScan</output_type>
-                <frame_name>lidar_link</frame_name>
-            </plugin>
-        </sensor>
-    </gazebo>
     <!-- imu -->
-    <joint name="imu_joint" type="fixed">
-        <parent link="base_link"/>
-        <child link="imu_link"/>
-        <origin xyz="${base_width/4} 0 ${(base_height+imu_height)/2}"/>
-    </joint>
-    <link name="imu_link">
-        <visual>
-            <geometry>
-                <box size="${imu_width} ${imu_depth} ${imu_height}"/>
-            </geometry>
-            <material name="purple" />
-        </visual>
-        <collision>
-            <geometry>
-                <box size="${imu_width} ${imu_depth} ${imu_height}"/>
-            </geometry>
-        </collision>
-        <xacro:box_inertia m="${imu_mass}" w="${imu_width}" d="${imu_depth}" h="${imu_height}" />
-    </link>
-    <gazebo reference="imu_link">
-        <material>Gazebo/Purple</material>
-        <sensor name="imu_sensor" type="imu">
-            <plugin filename="libgazebo_ros_imu_sensor.so" name="imu_plugin">
-                <ros>
-                    <namespace>/bot</namespace>
-                    <remapping>~/out:=imu</remapping>
-                </ros>
-                <initial_orientation_as_reference>false</initial_orientation_as_reference>
-            </plugin>
-            <always_on>true</always_on>
-            <update_rate>100</update_rate>
-            <visualize>true</visualize>
-            <imu>
-                <angular_velocity>
-                    <x>
-                        <noise type="gaussian">
-                            <mean>0.0</mean>
-                            <stddev>2e-4</stddev>
-                            <bias_mean>0.0000075</bias_mean>
-                            <bias_stddev>0.0000008</bias_stddev>
-                        </noise>
-                    </x>
-                    <y>
-                        <noise type="gaussian">
-                            <mean>0.0</mean>
-                            <stddev>2e-4</stddev>
-                            <bias_mean>0.0000075</bias_mean>
-                            <bias_stddev>0.0000008</bias_stddev>
-                        </noise>
-                    </y>
-                    <z>
-                        <noise type="gaussian">
-                            <mean>0.0</mean>
-                            <stddev>2e-4</stddev>
-                            <bias_mean>0.0000075</bias_mean>
-                            <bias_stddev>0.0000008</bias_stddev>
-                        </noise>
-                    </z>
-                </angular_velocity>
-                <linear_acceleration>
-                    <x>
-                        <noise type="gaussian">
-                            <mean>0.0</mean>
-                            <stddev>1.7e-2</stddev>
-                            <bias_mean>0.1</bias_mean>
-                            <bias_stddev>0.001</bias_stddev>
-                        </noise>
-                    </x>
-                    <y>
-                        <noise type="gaussian">
-                            <mean>0.0</mean>
-                            <stddev>1.7e-2</stddev>
-                            <bias_mean>0.1</bias_mean>
-                            <bias_stddev>0.001</bias_stddev>
-                        </noise>
-                    </y>
-                    <z>
-                        <noise type="gaussian">
-                            <mean>0.0</mean>
-                            <stddev>1.7e-2</stddev>
-                            <bias_mean>0.1</bias_mean>
-                            <bias_stddev>0.001</bias_stddev>
-                        </noise>
-                    </z>
-                </linear_acceleration>
-            </imu>
-        </sensor>
-    </gazebo>
-    <!-- differential_drive_controller plugin -->
-    <gazebo>
-        <plugin name="differential_drive_controller" filename="libgazebo_ros_diff_drive.so">
-            <ros>
-                <namespace>/bot</namespace>
-                <!-- <argument>cmd_vel:=cmd_demo</argument>
-                <argument>odom:=odom_demo</argument> -->
-            </ros>
-            <robot_base_frame>base_link</robot_base_frame>
-            <update_rate>100</update_rate>
-            <left_joint>left_wheel_joint</left_joint>
-            <right_joint>right_wheel_joint</right_joint>
-            <wheel_separation>0.26</wheel_separation>
-            <wheel_diameter>0.2</wheel_diameter>
-            <publish_odom>true</publish_odom>
-            <publish_odom_tf>false</publish_odom_tf>
-            <publish_wheel_tf>true</publish_wheel_tf>
-            <odometry_frame>odom</odometry_frame>
-            <max_wheel_torque>10</max_wheel_torque>
-            <!-- Wheel acceleration, in rad/s^2, defaults to 0.0 rad/s^2 -->
-            <max_acceleration>1.0</max_acceleration>
-        </plugin>
-    </gazebo>
+    <!-- <joint name="imu_joint" type="fixed"> -->
+    <!--     <parent link="base_link" /> -->
+    <!--     <child link="imu_link" /> -->
+    <!--     <origin xyz="${base_width/4} 0 ${(base_height+imu_height)/2}" /> -->
+    <!-- </joint> -->
+    <!---->
+    <!-- <link name="imu_link"> -->
+    <!--     <visual> -->
+    <!--         <geometry> -->
+    <!--             <box size="${imu_width} ${imu_depth} ${imu_height}" /> -->
+    <!--         </geometry> -->
+    <!--         <material name="purple" /> -->
+    <!--     </visual> -->
+    <!--     <collision> -->
+    <!--         <geometry> -->
+    <!--             <box size="${imu_width} ${imu_depth} ${imu_height}" /> -->
+    <!--         </geometry> -->
+    <!--     </collision> -->
+    <!--     <xacro:box_inertia m="${imu_mass}" w="${imu_width}" d="${imu_depth}" h="${imu_height}" /> -->
+    <!-- </link> -->
+    <!-- <gazebo reference="imu_link"> -->
+    <!--     <material>Gazebo/Purple</material> -->
+    <!--     <sensor name="imu_sensor" type="imu"> -->
+    <!--         <plugin filename="libgazebo_ros_imu_sensor.so" name="imu_plugin"> -->
+    <!--             <ros> -->
+    <!--                 <namespace>/bot</namespace> -->
+    <!--                 <remapping>~/out:=imu</remapping> -->
+    <!--             </ros> -->
+    <!--             <initial_orientation_as_reference>false</initial_orientation_as_reference> -->
+    <!--         </plugin> -->
+    <!--         <always_on>true</always_on> -->
+    <!--         <update_rate>100</update_rate> -->
+    <!--         <visualize>true</visualize> -->
+    <!--         <imu> -->
+    <!--             <angular_velocity> -->
+    <!--                 <x> -->
+    <!--                     <noise type="gaussian"> -->
+    <!--                         <mean>0.0</mean> -->
+    <!--                         <stddev>2e-4</stddev> -->
+    <!--                         <bias_mean>0.0000075</bias_mean> -->
+    <!--                         <bias_stddev>0.0000008</bias_stddev> -->
+    <!--                     </noise> -->
+    <!--                 </x> -->
+    <!--                 <y> -->
+    <!--                     <noise type="gaussian"> -->
+    <!--                         <mean>0.0</mean> -->
+    <!--                         <stddev>2e-4</stddev> -->
+    <!--                         <bias_mean>0.0000075</bias_mean> -->
+    <!--                         <bias_stddev>0.0000008</bias_stddev> -->
+    <!--                     </noise> -->
+    <!--                 </y> -->
+    <!--                 <z> -->
+    <!--                     <noise type="gaussian"> -->
+    <!--                         <mean>0.0</mean> -->
+    <!--                         <stddev>2e-4</stddev> -->
+    <!--                         <bias_mean>0.0000075</bias_mean> -->
+    <!--                         <bias_stddev>0.0000008</bias_stddev> -->
+    <!--                     </noise> -->
+    <!--                 </z> -->
+    <!--             </angular_velocity> -->
+    <!--             <linear_acceleration> -->
+    <!--                 <x> -->
+    <!--                     <noise type="gaussian"> -->
+    <!--                         <mean>0.0</mean> -->
+    <!--                         <stddev>1.7e-2</stddev> -->
+    <!--                         <bias_mean>0.1</bias_mean> -->
+    <!--                         <bias_stddev>0.001</bias_stddev> -->
+    <!--                     </noise> -->
+    <!--                 </x> -->
+    <!--                 <y> -->
+    <!--                     <noise type="gaussian"> -->
+    <!--                         <mean>0.0</mean> -->
+    <!--                         <stddev>1.7e-2</stddev> -->
+    <!--                         <bias_mean>0.1</bias_mean> -->
+    <!--                         <bias_stddev>0.001</bias_stddev> -->
+    <!--                     </noise> -->
+    <!--                 </y> -->
+    <!--                 <z> -->
+    <!--                     <noise type="gaussian"> -->
+    <!--                         <mean>0.0</mean> -->
+    <!--                         <stddev>1.7e-2</stddev> -->
+    <!--                         <bias_mean>0.1</bias_mean> -->
+    <!--                         <bias_stddev>0.001</bias_stddev> -->
+    <!--                     </noise> -->
+    <!--                 </z> -->
+    <!--             </linear_acceleration> -->
+    <!--         </imu> -->
+    <!--     </sensor> -->
+    <!-- </gazebo> -->
 </robot>
